File: priority_encoder/priority_encoder.sch (KiCad schematic (older format))
At the start: 44 parts, among them U1 plot_v1, U10 plot_v1, U11 plot_v1, U12 plot_v1, U13 adc_bridge_8, U14 plot_v1, U15 plot_v1, U16 plot_v1, U17 plot_v1, U18 plot_v1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

Commit message: Update priority_encoder.sch
Parts:
- removed R4: 1k, symbol resistor
- removed U12, U14, U15, U16, U17, U18, U19, U20, Ua1: plot_v1, symbol plot_v1
- removed U21: bala_priority_encoder, symbol bala_priority_encoder
- removed U22: dac_bridge_4, symbol dac_bridge_4
- removed U23: adc_bridge_8, symbol adc_bridge_8
- removed v10, v11, v12, v13, v14, v15, v16, v9: pulse, R1, symbol pulse
- added U12: priority_encode_vanshika, symbol priority_encode_vanshika
- added U14: dac_bridge_3, symbol dac_bridge_3
Connections:
- net at U13.10 (OUT2): now also U12.2 (i6)
- net at U13.11 (OUT3): now also U12.3 (i5)
- net at U13.12 (OUT4): now also U12.4 (i4)
- net at U13.13 (OUT5): now also U12.5 (i3)
- net at U13.14 (OUT6): now also U12.6 (i2)
- net at U13.15 (OUT7): now also U12.7 (i1)
- net at U13.16 (OUT8): now also U12.8 (i0)
- net at U13.9 (OUT1): now also U12.1 (i7)
- net at R1.1: now also U14.4 (OUT1)
- net at R2.1: now also U14.5 (OUT2)
- net at R3.1: now also U14.6 (OUT3)
- new net: U12.9 (o2), U14.1 (IN1)
- new net: U12.10 (o1), U14.2 (IN2)
- new net: U12.11 (o0), U14.3 (IN3)
Other:
- note added: "8x3 Priority Encoder Circuit"
- moved on the sheet: R1, R2, R3, U1, U10, U11, U13, U2, U3, U4, U5, U6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
